File: placas/MOD/mod-AD&DA/mod-AD-DA.sch (KiCad schematic (older format))
At the start: 19 parts, among them K1 jum_EN2, P1 FPGA, P1_IN FPGA, P2 IO aislados, U1 ISO7242A, U1 LP2951

Commit message: Primer version modulo AD&DA. para revision y correccion
Parts:
- removed P1_IN: FPGA, symbol CONN_5X2
- removed P2: IO aislados, symbol CONN_7
- removed U?: MAX681, symbol MAX681
- added BOR1: AN_IN, symbol CONN_2
- added BOR2: AUX1_OUT, symbol CONN_2
- added BOR3: AUX2_OUT, symbol CONN_2
- added BOR4: AN_OUT, symbol CONN_2
- added C10: 10 uF, symbol CAPAPOL
- added C11, C7, C8: 1uF, symbol C
- added C12, C13: 0.1uF, symbol C
- added C14: 10pF, symbol C
- added C9: 0.01uF, symbol CAPAPOL
- added JMP1, JMP3: SEL_ENT, symbol CONN_5X2
- added JMP2: SEL_ENT, symbol CONN_12X2
- added JMP4: SEL_ENT, symbol CONN_9X2
- added R10, R7, R9: 1k, symbol R
- added R5: 100k, symbol R
- added R6: 2k, symbol RVAR
- added R8: 1k2, symbol R
- added U2: ADCS7476, symbol ADCS7476
- added U3: MAX680, symbol MAX680
- added U4, U7: LM324, symbol LM324
- added U5: LP2951, symbol LP2951
- added U6: DAC121S101, symbol DAC121S101
- added U8: ISO7242A, symbol ISO7242A
- renumbered U1 to U9
Connections:
- net labels added: +VIN, +VOUT, A+, A-, AO, AO1 A, AO1 B, AO1 C, AO1 D, AO2 A, AO2 B, AO2 C, B+, B-, BIPOLAR, BO, C+, C-, CO, CS_ADC  <<, CS_ADC <<, CS_DAC  <<, CS_DAC <<, D+, D-, DATA     <<, DATA >>, DIRECTO, DO, SCLK    <<, SCLK <<, SDATA (IN DAC) <<, SDATA (OUT ADC) >>, UNIPOLAR, VREF ADC, VREF DAC
- wire segments 93 -> 312
- no-connect marks 6 -> 14
Other:
- note added: "ADC\n"
- note added: "AJUSTE VREF ADC"
- note added: "AJUSTE VREF DAC"
- note added: "BORNE ENTRADA\nCANAL ANALOGICO\n"
- note added: "BORNE SALIDA\nALIMENTACION\n AUXILIAR\n"
- note added: "BORNE SALIDA\nCANAL ANALOGICO\n"
- note added: "CONEXION CON\nPLACA PRINCIPAL\n"
- note added: "Conversor +5VCC A +/- 10 VCC.\nAlimentacion de Operacionales"
- note added: "DAC"
- note added: "El potenciometro R3 permite ajustar\n la tension de referencia en todo \nel rango del ADCS7476 (2,7 a 5,2 V)"
- note added: "El potenciometro R6 permite ajustar\n la tension de referencia en todo \nel rango del DAC121S101 (2,7 a 5,2 V)"
- note added: "JMP SELECCION\nENTRADA: \n/DIRECTA \n/ OPERACIONALES\n"
- note added: "JMP SELECCION\nSALIDA: \n/UNIPOLAR \n/ BIPOLAR \n/ OPERACIONALES\n"
- note added: "LOS TERMINALES DE LOS OPERACIONALES ESTAN EN BORNES HEMBRA\nPARA PERMITIR AL USUARIO HACER CONEXIONES ENTRE ELLOS. \nMEDIANTE JMP1 SELECCIONAR LA SALIDA DE ALGUN OA (U4) COMO ENTRADA DEL ADC.\nMEDIANTE JMP3 SELECCIONAR LA SALIDA DE ALGUN OA (U7) COMO SALIDA DEL DAC"
- note added: "OPERACIONALES EN BORNES:"
- note added: "PINES HEMBRA \nCONEXIONADO\nOPERACIONALES\nADC\n"
- note added: "PINES HEMBRA \nCONEXIONADO\nOPERACIONALES\nDAC\n"
- note added: "SALIDA BIPOLAR +/- VREF"
- note added: "TIPO: LMC6484 (IN/OUT RAIL2RAIL) PIN COMPATIBLE CON LM324, ETC. DIP C/ ZOCALO"
- moved on the sheet: C1, C2, C3, C4, C5, C6, K1, P1, R1, R2, R3, R4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
