File: placas/MOD/mod-AD&DA/mod-AD-DA-1.sch (KiCad schematic (older format))
At the start: 44 parts, among them P1 FPGA, U1 LP2951, U2 NJU7201, U3 MAX871, U4 LP2950, U5 AD5160, U6 ADC124S101, U7 DAC124S085, U8 TS924

Commit message: 
Parts:
- removed C1reg1: 0.33uF, symbol C
- removed C2reg1, C2reg2: 3.3 uF, symbol CAPAPOL
- removed Cpot3: 0.1uF, symbol C
- removed Cpot7, Cpot8: 1uF, symbol C
- removed U2: NJU7201, symbol NJU7201
- removed U4: LP2950, symbol LP2950
- added C2U1: 3.3uF, symbol C
- added U2: NJM78L06A, symbol NJM78L06A
- added U4: NJM78L05A, symbol NJM78L05A
- C1U2: renamed from Cpot5; value 0.1uF -> 0.33uF
- C1U7: renamed from C4; value 0.33uF -> 10uF
- C2U4: renamed from Cpot4; value 1uF -> 0.1uF
- renumbered C14 to C1AU8, C5 to C1BU8, C7 to C1CU8, C8 to C1DU8, C6 to C1U3, C1reg2 to C1U4, Cpot1 to C1U5, Cpot6 to C2U2, C3 to C2U3, Cpot2 to C2U5, C1 to C2U7, C2 to C3U3, Cbypass1 to Cbypass1U5, R1A1 to R1AU1, R9 to R1AU8, R1 to R1BU8, R3 to R1CU8, R5 to R1DU8, R10 to R2AU8, R6 to R2BU8, R7 to R2CU8, R8 to R2DU8, R2 to R2U1, R4 to R3U1
Connections:
- net +5VA: now also U4.1 (OUT)
- net GND: now also C2U1.2, U2.2 (GND), U4.2 (GND)
- net VAA: now also C1U5.1, C2U5.1, U5.2 (VDD), C2U1.1
- net VCC: now also U2.3 (IN), U4.3 (IN)
- removed net +5V: C1U5.1, C2U2.1, C2U5.1, U1.8 (INPUT), U5.2 (VDD)
- new net +6V: C2U2.1, U1.8 (INPUT), U2.1 (OUT)
Other:
- note added: "+6V"
- note added: "El potenciometro digital R1 (entre W y B de U5), \nen conjunto con R1A y R2 \npermite ajustar la tension de referencia \nen todo el rango del ADC (2,7 a 5,2 5V)\nR1 nominal 10K\nR1 min = 60 @ DATAIN = 0x00\nR1 max = 9960 @ DATAIN = 0xFF"
- note added: "Estos circuitos permiten\n la salida Bipolar de cada canal\n"
- note removed: "+5,2V"
- note removed: "El potenciometro digital R1 (entre W y B), \nen conjunto con R1A y R2 \npermite ajustar la tension de referencia \nen todo el rango del ADC (2,7 a 5,2 5V)\nR1 nominal 10K\nR1 min = 60 @ DATAIN = 0x00\nR1 max = 9960 @ DATAIN = 0xFF"
- note removed: "TANTALIO \nO ELECTROLITICO"
- moved on the sheet: C1U2, C1U5, C2U2, C2U5
